Commit message: added ability to spawn sdf

File: src/healthbot/urdf/hbot_base.xacro (robot description, xacro)
@@ -2,27 +2,27 @@
 <robot name="hbot" xmlns:xacro="http://www.ros.org/wiki/xacro">
 <!-- Chassis vars -->
-<xacro:property name="chassis_xyz" value="0.0 0.0 0.1"/>
-<xacro:property name="chassis_rpy" value="0.0 0.0 0.0"/>
-<xacro:property name="chassis_visual_xyz" value="0.0 0.0 0.0"/>
+<xacro:property name="chassis_xyz" value="-0.1 0 -0.1"/>
+<xacro:property name="chassis_rpy" value="0 0 0"/>
+<xacro:property name="chassis_visual_xyz" value="-0.1 0 -0.1"/>
 <!-- Caster wheel vars -->
-<xacro:property name="caster_xyz" value="0.35 0.0 -0.05"/>
+<xacro:property name="caster_xyz" value="-0.8 0 -0.125"/>
 <xacro:property name="caster_rpy" value="0 0 0"/>
-<xacro:property name="castor_wheel_size" value="0.06"/>
-<xacro:property name="visual_caster_xyz" value="0.2 0.0 -0.05"/>
+<xacro:property name="castor_wheel_size" value="0.125"/>
+<xacro:property name="visual_caster_xyz" value="-0.8 0 -0.125"/>
 <!-- Side wheels -->
-<xacro:property name="side_wheel_length" value="0.04"/>
-<xacro:property name="side_wheel_radius" value="0.1"/>
+<xacro:property name="side_wheel_length" value="0.05"/>
+<xacro:property name="side_wheel_radius" value="0.125"/>
 <xacro:property name="side_wheel_mass" value="0.2"/>
 <xacro:property name="axis_xyz" value="0 1 0"/>
 <xacro:property name="axis_rpy" value="0 0 0"/>
 <!-- Right wheel info -->
-<xacro:property name="right_xyz" value="0 0 0"/>
+<xacro:property name="right_xyz" value="0.8 -0.535 0.125"/>
 <xacro:property name="right_rpy" value="0 1.57 1.57"/>
-<xacro:property name="joint_right_xpy" value="-0.05 0.15 0.0"/>
+<xacro:property name="joint_right_xpy" value="0 0 0.03"/>
 <xacro:property name="joint_right_rpy" value="0 0 0"/>
 <!-- Left wheel info -->
-<xacro:property name="left_xyz" value="0 0 0"/>
+<xacro:property name="left_xyz" value="0.8 0.535 0.125"/>
 <xacro:property name="left_rpy" value="0 1.57 1.57"/>
-<xacro:property name="joint_left_xpy" value="-0.05 -0.15 0.0"/>
+<xacro:property name="joint_left_xpy" value="-0 0 -0.03"/>
 <xacro:property name="joint_left_rpy" value="0.0 0.0 0.0"/>
 <!-- imports -->
@@ -32,107 +32,239 @@
   <joint name="fixed" type="fixed">
     <parent link="world"/>
-    <child link="chassis"/>
+    <child link="mobile_base__chassis"/>
   </joint>
 <!-- Chassis and front wheel -->
-  <link name='chassis'>
-    <pose>0 0 0.1 0 0 0</pose>
-    <inertial>
-      <origin xyz="${chassis_xyz}" rpy="${chassis_rpy}"/>
-      <mass value="4.0"/>
-      <inertia ixx="0.0395416666667" ixy="0" ixz="0" iyy="0.106208333333" iyz="0" izz="0.106208333333"/>
-    </inertial>
-    <collision name="chassis_collision">
-      <origin xyz="${chassis_xyz}" rpy="${chassis_rpy}"/>
-     <geometry>
-       <box size="0.50 0.30 0.07"/>
-     </geometry>
-    </collision>
-    <visual>
-      <origin xyz="${chassis_visual_xyz}" rpy="${chassis_rpy}"/>
-      <geometry>
-        <box size="0.50 0.30 0.07"/>
-      </geometry>
-      <material name="red"/>
-    </visual>
-  <!-- Caster wheel -->
-    <collision>
-      <origin xyz="${caster_xyz}" rpy="${caster_rpy}"/>
-      <geometry>
-        <sphere radius="${castor_wheel_size}"/>
-      </geometry>
-      <surface>
-        <friction>
-          <ode>
-            <mu>0</mu>
-            <mu2>0</mu2>
-            <slip1>1.0</slip1>
-            <slip2>1.0</slip2>
-          </ode>
-        </friction>
-      </surface>
-    </collision>
-    <visual>
-      <origin xyz="${caster_xyz}" rpy="${caster_rpy}"/>
-      <geometry>
-        <sphere radius="${castor_wheel_size}"/>
-      </geometry>
-    </visual>
-  </link>
-  <!-- wheels -->
-  <link name="right_wheel">
-    <inertial>
-      <origin xyz="${right_xyz}" rpy="${right_rpy}"/>
-      <mass value="${side_wheel_mass}"/>
-      <inertia ixx="0.0005267" ixy="0.0" ixz="0.0" iyy="0.00053" iyz="0.0" izz="0.001"/>
-    </inertial>
-    <visual>
-      <origin xyz="${right_xyz}" rpy="${right_rpy}"/>
-      <geometry>
-        <cylinder radius="${side_wheel_radius}" length="${side_wheel_length}"/>
-      </geometry>
-      <material name="black"/>
-    </visual>
-    <collision>
-      <origin xyz="${right_xyz}" rpy="${right_rpy}"/>
-      <geometry>
-        <cylinder radius="${side_wheel_radius}" length="${side_wheel_length}"/>
-      </geometry>
-    </collision>
-  </link>
-   <link name="left_wheel">
-    <inertial>
-      <origin xyz="${left_xyz}" rpy="${left_rpy}"/>
-      <mass value="${side_wheel_mass}"/>
-      <inertia ixx="0.0005267" ixy="0.0" ixz="0.0" iyy="0.00053" iyz="0.0" izz="0.001"/>
-    </inertial>
-    <visual>
-      <origin xyz="${left_xyz}" rpy="${left_rpy}"/>
-      <geometry>
-        <cylinder radius="${side_wheel_radius}" length="${side_wheel_length}"/>
-      </geometry>
-      <material name="black"/>
-    </visual>
-    <collision>
-      <origin xyz="${left_xyz}" rpy="${left_rpy}"/>
-      <geometry>
-        <cylinder radius="${side_wheel_radius}" length="${side_wheel_length}"/>
-      </geometry>
-    </collision>
-  </link>
-  <joint name="joint_left_wheel" type="continuous">
-    <origin xyz="${left_xyz}" rpy="${left_rpy}"/>
-    <parent link="chassis"/>
-    <child link="left_wheel"/>
-    <axis xyz="${axis_xyz}" rpy='${axis_rpy}'/>
-    <limit effort="10000.0" velocity="1000.0"/>
-    <joint_properties damping='1.0' friction='1.0'/>
-  </joint>
-  <joint name="joint_right_wheel" type="continuous">
-    <origin xyz="${right_xyz}" rpy="${right_rpy}"/>
-    <parent link="chassis"/>
-    <child link="right_wheel"/>
-    <axis xyz="${axis_xyz}" rpy='${axis_rpy}'/>
-    <limit effort="10000.0" velocity="1000.0"/>
-    <joint_properties damping='1.0' friction='1.0'/>
-  </joint>
+  <joint name="mobile_base__left_wheel_hinge" type="fixed">
+    <parent link="mobile_base__chassis"/>
+    <child link="mobile_base__left_wheel"/>
+    <origin xyz="0.79999 0.505   0.12499" rpy="0     1.5707 1.5707"/>
+    <axis xyz="9.e-05 9.e-05 1.e+00"/>
+    <limit lower="0" upper="0" effort="0" velocity="0"/>
+  </joint>
+  <joint name="mobile_base__right_wheel_hinge" type="fixed">
+    <parent link="mobile_base__chassis"/>
+    <child link="mobile_base__right_wheel"/>
+    <origin xyz="0.8   -0.505  0.125" rpy="0     1.5707 1.5707"/>
+    <axis xyz="9.e-05 9.e-05 1.e+00"/>
+    <limit lower="0" upper="0" effort="0" velocity="0"/>
+  </joint>
+  <link name="mobile_base__chassis">
+    <inertial>
+      <mass value="20.0"/>
+      <origin xyz="-0.1  0  -0.1" rpy="0 0 0"/>
+      <inertia ixx="0.5" ixy="0" ixz="0" iyy="1.0" iyz="0" izz="0.1"/>
+    </inertial>
+    <collision name="mobile_base__collision">
+      <origin xyz="0   0   0.25" rpy="0 0 0"/>
+      <geometry>
+        <box size="2 1 0.3"/>
+      </geometry>
+    </collision>
+    <collision name="mobile_base__caster_collision">
+      <origin xyz="-0.8    0     0.125" rpy="0 0 0"/>
+      <geometry>
+        <sphere radius=".125"/>
+      </geometry>
+    </collision>
+    <visual name="mobile_base__visual">
+      <origin xyz="0   0   0.25" rpy="0 0 0"/>
+      <geometry>
+        <box size="2 1 0.3"/>
+      </geometry>
+    </visual>
+    <visual name="mobile_base__caster_visual">
+      <origin xyz="-0.8    0     0.125" rpy="0 0 0"/>
+      <geometry>
+        <sphere radius=".125"/>
+      </geometry>
+    </visual>
+  </link>
+  <link name="mobile_base__left_wheel">
+    <inertial>
+      <mass value="0"/>
+      <origin xyz="0 0 0" rpy="0 0 0"/>
+      <inertia ixx="0" ixy="0" ixz="0" iyy="0" iyz="0" izz="0"/>
+    </inertial>
+    <collision name="mobile_base__collision">
+      <origin xyz="0   0   0.03" rpy="0 0 0"/>
+      <geometry>
+        <cylinder radius=".125" length=".05"/>
+      </geometry>
+    </collision>
+    <visual name="mobile_base__visual">
+      <origin xyz="0   0   0.03" rpy="0 0 0"/>
+      <geometry>
+        <cylinder radius=".125" length=".05"/>
+      </geometry>
+    </visual>
+  </link>
+  <link name="mobile_base__right_wheel">
+    <inertial>
+      <mass value="0"/>
+      <origin xyz="0 0 0" rpy="0 0 0"/>
+      <inertia ixx="0" ixy="0" ixz="0" iyy="0" iyz="0" izz="0"/>
+    </inertial>
+    <collision name="mobile_base__collision">
+      <origin xyz="0    0   -0.03" rpy="0 0 0"/>
+      <geometry>
+        <cylinder radius=".125" length=".05"/>
+      </geometry>
+    </collision>
+    <visual name="mobile_base__visual">
+      <origin xyz="0    0   -0.03" rpy="0 0 0"/>
+      <geometry>
+        <cylinder radius=".125" length=".05"/>
+      </geometry>
+    </visual>
+  </link>
+ <!-- Gripper -->
+ <joint name="simple_gripper__palm_left_finger" type="revolute">
+    <parent link="simple_gripper__palm"/>
+    <child link="simple_gripper__left_finger"/>
+    <origin xyz="-0.00606  0.09393  0" rpy="0       0      -0.78539"/>
+    <axis xyz="0 0 1"/>
+    <limit lower="-0.4" upper="0.4" effort="0.0" velocity="0.0"/>
+  </joint>
+  <joint name="simple_gripper__left_finger_tip" type="revolute">
+    <parent link="simple_gripper__left_finger"/>
+    <child link="simple_gripper__left_finger_tip"/>
+    <origin xyz="0.02545 0.31688 0" rpy="0      0      2.35609"/>
+    <axis xyz="0 0 1"/>
+    <limit lower="-0.4" upper="0.4" effort="0.0" velocity="0.0"/>
+  </joint>
+  <joint name="simple_gripper__palm_right_finger" type="revolute">
+    <parent link="simple_gripper__palm"/>
+    <child link="simple_gripper__right_finger"/>
+    <origin xyz="-0.00606 -0.09393  0" rpy="0      0      0.78539"/>
+    <axis xyz="0 0 1"/>
+    <limit lower="-0.4" upper="0.4" effort="0.0" velocity="0.0"/>
+  </joint>
+  <joint name="simple_gripper__right_finger_tip" type="revolute">
+    <parent link="simple_gripper__right_finger"/>
+    <child link="simple_gripper__right_finger_tip"/>
+    <origin xyz="0.02546 -0.31687  0" rpy="0      0      0.78531"/>
+    <axis xyz="0 0 1"/>
+    <limit lower="-0.4" upper="0.4" effort="0.0" velocity="0.0"/>
+  </joint>
+  <joint name="simple_gripper__palm_riser" type="prismatic">
+    <parent link="simple_gripper__riser"/>
+    <child link="simple_gripper__palm"/>
+    <origin xyz="0   0   0.05" rpy="0 0 0"/>
+    <axis xyz="0 0 1"/>
+    <limit lower="0.0" upper="0.9" effort="0.0" velocity="0.0"/>
+  </joint>
+  <link name="simple_gripper__riser">
+    <inertial>
+      <mass value="10.0"/>
+      <origin xyz="0   0  -0.5" rpy="0 0 0"/>
+      <inertia ixx="0.01" ixy="0" ixz="0" iyy="0.01" iyz="0" izz="0.01"/>
+    </inertial>
+    <collision name="simple_gripper__collision">
+      <origin xyz="-0.15  0    0.5" rpy="0 0 0"/>
+      <geometry>
+        <box size="0.2 0.2 1.0"/>
+      </geometry>
+    </collision>
+    <visual name="simple_gripper__visual">
+      <origin xyz="-0.15  0    0.5" rpy="0 0 0"/>
+      <geometry>
+        <box size="0.2 0.2 1.0"/>
+      </geometry>
+    </visual>
+  </link>
+  <link name="simple_gripper__palm">
+    <inertial>
+      <mass value="0.5"/>
+      <origin xyz="0 0 0" rpy="0 0 0"/>
+      <inertia ixx="0.01" ixy="0" ixz="0" iyy="0.01" iyz="0" izz="0.01"/>
+    </inertial>
+    <collision name="simple_gripper__collision">
+      <origin xyz="0 0 0" rpy="0 0 0"/>
+      <geometry>
+        <box size="0.1 0.2 0.1"/>
+      </geometry>
+    </collision>
+    <visual name="simple_gripper__visual">
+      <origin xyz="0 0 0" rpy="0 0 0"/>
+      <geometry>
+        <box size="0.1 0.2 0.1"/>
+      </geometry>
+    </visual>
+  </link>
+  <link name="simple_gripper__left_finger">
+    <inertial>
+      <mass value="0.1"/>
+      <origin xyz="0 0 0" rpy="0 0 0"/>
+      <inertia ixx="0.01" ixy="0" ixz="0" iyy="0.01" iyz="0" izz="0.01"/>
+    </inertial>
+    <collision name="simple_gripper__collision">
+      <origin xyz="0   0.15 0" rpy="0 0 0"/>
+      <geometry>
+        <box size="0.1 0.3 0.1"/>
+      </geometry>
+    </collision>
+    <visual name="simple_gripper__visual">
+      <origin xyz="0   0.15 0" rpy="0 0 0"/>
+      <geometry>
+        <box size="0.1 0.3 0.1"/>
+      </geometry>
+    </visual>
+  </link>
+  <link name="simple_gripper__left_finger_tip">
+    <inertial>
+      <mass value="0.1"/>
+      <origin xyz="0 0 0" rpy="0 0 0"/>
+      <inertia ixx="0.01" ixy="0" ixz="0" iyy="0.01" iyz="0" izz="0.01"/>
+    </inertial>
+    <collision name="simple_gripper__collision">
+      <origin xyz="0  -0.1  0" rpy="0 0 0"/>
+      <geometry>
+        <box size="0.1 0.2 0.1"/>
+      </geometry>
+    </collision>
+    <visual name="simple_gripper__visual">
+      <origin xyz="0  -0.1  0" rpy="0 0 0"/>
+      <geometry>
+        <box size="0.1 0.2 0.1"/>
+      </geometry>
+    </visual>
+  </link>
+  <link name="simple_gripper__right_finger">
+    <inertial>
+      <mass value="0.1"/>
+      <origin xyz="0 0 0" rpy="0 0 0"/>
+      <inertia ixx="0.01" ixy="0" ixz="0" iyy="0.01" iyz="0" izz="0.01"/>
+    </inertial>
+    <collision name="simple_gripper__collision">
+      <origin xyz="0   -0.15  0" rpy="0 0 0"/>
+      <geometry>
+        <box size="0.1 0.3 0.1"/>
+      </geometry>
+    </collision>
+    <visual name="simple_gripper__visual">
+      <origin xyz="0   -0.15  0" rpy="0 0 0"/>
+      <geometry>
+        <box size="0.1 0.3 0.1"/>
+      </geometry>
+    </visual>
+  </link>
+  <link name="simple_gripper__right_finger_tip">
+    <inertial>
+      <mass value="0.1"/>
+      <origin xyz="0 0 0" rpy="0 0 0"/>
+      <inertia ixx="0.01" ixy="0" ixz="0" iyy="0.01" iyz="0" izz="0.01"/>
+    </inertial>
+    <collision name="simple_gripper__collision">
+      <origin xyz="0  -0.1  0" rpy="0 0 0"/>
+      <geometry>
+        <box size="0.1 0.2 0.1"/>
+      </geometry>
+    </collision>
+    <visual name="simple_gripper__visual">
+      <origin xyz="0  -0.1  0" rpy="0 0 0"/>
+      <geometry>
+        <box size="0.1 0.2 0.1"/>
+      </geometry>
+    </visual>
+  </link>
 </robot>
