Commit message: made wheels move

File: src/healthbot/urdf/healthbot.xacro (robot description, xacro)
@@ -1,4 +1,6 @@
 <?xml version="1.0" ?>
-<robot name="healthbot">
+<robot name="healthbot" xmlns:xacro="http://www.ros.org/wiki/xacro">
+  <xacro:include filename="$(find healthbot)/urdf/gazebo.xacro" />
+  <xacro:include filename="$(find healthbot)/urdf/transmission.xacro" />
   <!-- Root link -->
 <link name="world"/>
@@ -7,94 +9,4 @@
   <child link="healthbot__chassis"/>
 </joint>
-<gazebo>
-  <plugin name="gazebo_ros_control" filename="libgazebo_ros_control.so">
-    <robotNamespace>/healthbot</robotNamespace>
-    <robotSimType>gazebo_ros_control/DefaultRobotHWSim</robotSimType>
-  </plugin>
-</gazebo>
-<transmission name="tran1">
-  <type>transmission_interface/SimpleTransmission</type>
-  <joint name="healthbot__palm_riser">
-    <hardwareInterface>hardware_interface/EffortJointInterface</hardwareInterface>
-  </joint>
-  <actuator name="motor1">
-    <hardwareInterface>hardware_interface/EffortJointInterface</hardwareInterface>
-    <mechanicalReduction>1</mechanicalReduction>
-  </actuator>
-</transmission>
-<transmission name="tran2">
-  <type>transmission_interface/SimpleTransmission</type>
-  <joint name="healthbot__joint_right_finger">
-    <hardwareInterface>hardware_interface/EffortJointInterface</hardwareInterface>
-  </joint>
-  <actuator name="motor2">
-    <hardwareInterface>hardware_interface/EffortJointInterface</hardwareInterface>
-    <mechanicalReduction>1</mechanicalReduction>
-  </actuator>
-</transmission>
-<transmission name="tran3">
-  <type>transmission_interface/SimpleTransmission</type>
-  <joint name="healthbot__joint_right_finger_tip">
-    <hardwareInterface>hardware_interface/EffortJointInterface</hardwareInterface>
-  </joint>
-  <actuator name="motor3">
-    <hardwareInterface>hardware_interface/EffortJointInterface</hardwareInterface>
-    <mechanicalReduction>1</mechanicalReduction>
-  </actuator>
-</transmission>
-<transmission name="tran4">
-  <type>transmission_interface/SimpleTransmission</type>
-  <joint name="healthbot__joint_left_finger">
-    <hardwareInterface>hardware_interface/EffortJointInterface</hardwareInterface>
-  </joint>
-  <actuator name="motor4">
-    <hardwareInterface>hardware_interface/EffortJointInterface</hardwareInterface>
-    <mechanicalReduction>1</mechanicalReduction>
-  </actuator>
-</transmission>
-<transmission name="tran5">
-  <type>transmission_interface/SimpleTransmission</type>
-  <joint name="healthbot__joint_left_finger_tip">
-    <hardwareInterface>hardware_interface/EffortJointInterface</hardwareInterface>
-  </joint>
-  <actuator name="motor5">
-    <hardwareInterface>hardware_interface/EffortJointInterface</hardwareInterface>
-    <mechanicalReduction>1</mechanicalReduction>
-  </actuator>
-</transmission>
-<transmission name="tran6">
-  <type>transmission_interface/SimpleTransmission</type>
-  <joint name="healthbot__right_wheel_hinge">
-    <hardwareInterface>hardware_interface/EffortJointInterface</hardwareInterface>
-  </joint>
-  <actuator name="motor6">
-    <hardwareInterface>hardware_interface/EffortJointInterface</hardwareInterface>
-    <mechanicalReduction>1</mechanicalReduction>
-  </actuator>
-</transmission>
-<transmission name="tran7">
-  <type>transmission_interface/SimpleTransmission</type>
-  <joint name="healthbot__left_wheel_hinge">
-    <hardwareInterface>hardware_interface/EffortJointInterface</hardwareInterface>
-  </joint>
-  <actuator name="motor7">
-    <hardwareInterface>hardware_interface/EffortJointInterface</hardwareInterface>
-    <mechanicalReduction>1</mechanicalReduction>
-  </actuator>
-</transmission>
-  <joint name="healthbot__chassis_gripper_fixed_joint" type="fixed">
-    <parent link="healthbot__chassis"/>
-    <child link="healthbot__riser"/>
-    <origin xyz="-1.09676  0       0.58693" rpy="0       0      -3.13784"/>
-    <axis xyz="0 0 0"/>
-    <limit lower="0" upper="0" effort="0" velocity="0"/>
-  </joint>
-  <joint name="healthbot__joint_left_finger_tip" type="revolute">
-    <parent link="healthbot__left_finger"/>
-    <child link="healthbot__left_finger_tip"/>
-    <origin xyz="-0.04411  0.31132 -0.00252" rpy="0       0      -2.62881"/>
-    <axis xyz="0 0 1"/>
-    <limit lower="-0.4" upper="0.4" effort="-1.0" velocity="-1.0"/>
-  </joint>
   <joint name="healthbot__left_wheel_hinge" type="revolute">
     <parent link="healthbot__chassis"/>
@@ -103,32 +15,4 @@
     <axis xyz="9.e-05 9.e-05 1.e+00"/>
     <limit lower="-1e+16" upper="1e+16" effort="-1.0" velocity="-1.0"/>
-  </joint>
-  <joint name="healthbot__joint_left_finger" type="revolute">
-    <parent link="healthbot__palm"/>
-    <child link="healthbot__left_finger"/>
-    <origin xyz="0.07149 -0.05105 -0.01288" rpy="0       0      -2.16075"/>
-    <axis xyz="0 0 1"/>
-    <limit lower="-0.4" upper="0.4" effort="-1.0" velocity="-1.0"/>
-  </joint>
-  <joint name="healthbot__joint_right_finger" type="revolute">
-    <parent link="healthbot__palm"/>
-    <child link="healthbot__right_finger"/>
-    <origin xyz="0.07084  0.05881 -0.01264" rpy="0      0      2.08708"/>
-    <axis xyz="0 0 1"/>
-    <limit lower="-0.4" upper="0.4" effort="-1.0" velocity="-1.0"/>
-  </joint>
-  <joint name="healthbot__palm_riser" type="prismatic">
-    <parent link="healthbot__riser"/>
-    <child link="healthbot__palm"/>
-    <origin xyz="1.2773e-01 -3.8000e-04 -4.3013e-01" rpy="0       0      -0.01002"/>
-    <axis xyz="0 0 1"/>
-    <limit lower="0.0" upper="0.9" effort="-1.0" velocity="-1.0"/>
-  </joint>
-  <joint name="healthbot__joint_right_finger_tip" type="revolute">
-    <parent link="healthbot__right_finger"/>
-    <child link="healthbot__right_finger_tip"/>
-    <origin xyz="-0.02849 -0.31307 -0.00111" rpy="0       0      -0.52322"/>
-    <axis xyz="0 0 1"/>
-    <limit lower="-0.4" upper="0.4" effort="-1.0" velocity="-1.0"/>
   </joint>
   <joint name="healthbot__right_wheel_hinge" type="revolute">
@@ -170,42 +54,4 @@
     </visual>
   </link>
-  <link name="healthbot__left_finger">
-    <inertial>
-      <mass value="0.1"/>
-      <origin xyz="0 0 0" rpy="0 0 0"/>
-      <inertia ixx="0.01" ixy="0" ixz="0" iyy="0.01" iyz="0" izz="0.01"/>
-    </inertial>
-    <collision name="healthbot__collision">
-      <origin xyz="0   0.15 0" rpy="0 0 0"/>
-      <geometry>
-        <box size="0.1 0.3 0.1"/>
-      </geometry>
-    </collision>
-    <visual name="healthbot__visual">
-      <origin xyz="0   0.15 0" rpy="0 0 0"/>
-      <geometry>
-        <box size="0.1 0.3 0.1"/>
-      </geometry>
-    </visual>
-  </link>
-  <link name="healthbot__left_finger_tip">
-    <inertial>
-      <mass value="0.1"/>
-      <origin xyz="0 0 0" rpy="0 0 0"/>
-      <inertia ixx="0.01" ixy="0" ixz="0" iyy="0.01" iyz="0" izz="0.01"/>
-    </inertial>
-    <collision name="healthbot__collision">
-      <origin xyz="0  -0.1  0" rpy="0 0 0"/>
-      <geometry>
-        <box size="0.1 0.2 0.1"/>
-      </geometry>
-    </collision>
-    <visual name="healthbot__visual">
-      <origin xyz="0  -0.1  0" rpy="0 0 0"/>
-      <geometry>
-        <box size="0.1 0.2 0.1"/>
-      </geometry>
-    </visual>
-  </link>
   <link name="healthbot__left_wheel">
     <inertial>
@@ -214,5 +60,5 @@
       <inertia ixx="1" ixy="0" ixz="0" iyy="1" iyz="0" izz="1"/>
     </inertial>
-    <collision name="healthbot__collision">
+    <collision>
       <origin xyz="0   0   0.03" rpy="0 0 0"/>
       <geometry>
@@ -220,5 +66,5 @@
       </geometry>
     </collision>
-    <visual name="healthbot__visual">
+    <visual >
       <origin xyz="0   0   0.03" rpy="0 0 0"/>
       <geometry>
@@ -227,12 +73,12 @@
     </visual>
   </link>
-  <link name="healthbot__palm">
+  <!-- <link name="healthbot__palm">
     <inertial>
       <mass value="0.5"/>
-      <origin xyz="0 0 0" rpy="0 0 0"/>
+      <origin xyz="0 0 0.3" rpy="0 0 0"/>
       <inertia ixx="0.01" ixy="0" ixz="0" iyy="0.01" iyz="0" izz="0.01"/>
     </inertial>
-    <collision name="healthbot__collision">
-      <origin xyz="0 0 0" rpy="0 0 0"/>
+    <collision >
+      <origin xyz="0 0 0.3" rpy="0 0 0"/>
       <geometry>
         <box size="0.1 0.2 0.1"/>
@@ -240,5 +86,5 @@
     </collision>
     <visual name="healthbot__visual">
-      <origin xyz="0 0 0" rpy="0 0 0"/>
+      <origin xyz="0 0 0.3" rpy="0 0 0"/>
       <geometry>
         <box size="0.1 0.2 0.1"/>
@@ -283,5 +129,5 @@
       </geometry>
     </visual>
-  </link>
+  </link> -->
   <link name="healthbot__right_wheel">
     <inertial>
@@ -303,5 +149,5 @@
     </visual>
   </link>
-  <link name="healthbot__riser">
+  <!-- <link name="healthbot__riser">
     <inertial>
       <mass value="10"/>
@@ -321,4 +167,4 @@
       </geometry>
     </visual>
-  </link>
+  </link> -->
 </robot>
