Commit message: made the wheel drive move the bot

File: src/healthbot/urdf/gazebo.xacro (robot description, xacro)
@@ -9,7 +9,11 @@
     <gazebo reference="healthbot__left_wheel">
         <material>Gazebo/Black</material>
+        <mu1>100.0</mu1>
+        <mu2>50.0</mu2>
     </gazebo>
     <gazebo reference="healthbot__right_wheel">
         <material>Gazebo/Black</material>
+        <mu1>100.0</mu1>
+        <mu2>50.0</mu2>
     </gazebo>
     <gazebo>
@@ -22,5 +26,5 @@
             <wheelSeparation>0.5380</wheelSeparation>
             <!-- Diameter of the wheels, in meters, defaults to 0.15 m -->
-            <wheelDiameter>0.25</wheelDiameter>
+            <wheelDiameter>0.4</wheelDiameter>
             <!-- Wheel acceleration, in rad/s^2, defaults to 0.0 rad/s^2 -->
             <wheelAcceleration>1.0</wheelAcceleration>

File: src/healthbot/urdf/healthbot.xacro (robot description, xacro)
@@ -3,10 +3,11 @@
   <xacro:include filename="$(find healthbot)/urdf/gazebo.xacro" />
   <xacro:include filename="$(find healthbot)/urdf/transmission.xacro" />
+  <xacro:property name="wheel_radius" value="0.2"/>
   <!-- Root link -->
-<link name="world"/>
+<!-- <link name="world"/>
 <joint name="fixed" type="fixed">
   <parent link="world"/>
   <child link="healthbot__chassis"/>
-</joint>
+</joint> -->
   <joint name="healthbot__left_wheel_hinge" type="revolute">
     <parent link="healthbot__chassis"/>
@@ -63,5 +64,5 @@
       <origin xyz="0   0   0.03" rpy="0 0 0"/>
       <geometry>
-        <cylinder radius="0.125" length="0.05"/>
+        <cylinder radius="${wheel_radius}" length="0.05"/>
       </geometry>
     </collision>
@@ -69,5 +70,5 @@
       <origin xyz="0   0   0.03" rpy="0 0 0"/>
       <geometry>
-        <cylinder radius="0.125" length="0.05"/>
+        <cylinder radius="${wheel_radius}" length="0.05"/>
       </geometry>
     </visual>
@@ -139,5 +140,5 @@
       <origin xyz="0    0   -0.03" rpy="0 0 0"/>
       <geometry>
-        <cylinder radius="0.125" length="0.05"/>
+        <cylinder radius="${wheel_radius}" length="0.05"/>
       </geometry>
     </collision>
@@ -145,5 +146,5 @@
       <origin xyz="0    0   -0.03" rpy="0 0 0"/>
       <geometry>
-        <cylinder radius="0.125" length="0.05"/>
+        <cylinder radius="${wheel_radius}" length="0.05"/>
       </geometry>
     </visual>
